File: HARDWARE/tiny_pov_arm/tiny_pov_arm.kicad_pcb (KiCad board)
At the start: 2 copper layers, 17 parts, among them J1 Conn_01x02_Socket, U1 AH1806W, U2 STM32G030J6Mx

Commit message: Completed V1 arm board layout
Parts:
- added BR1: DBF310-13, tiny_pov_footprints:DBF_DIO, F.Cu at (146.9, 102.6)
- added C3: 22 uF, tiny_pov_footprints:C_0603_hand_solder, F.Cu at (160.3, 100.0)
- added C4: 22 uF, tiny_pov_footprints:C_0603_hand_solder, F.Cu at (156.6, 100.0)
- added C5: 100 uF, tiny_pov_footprints:C_polarized_TH, B.Cu at (153.4, 107.3)
- added C6: 100 nF, tiny_pov_footprints:C_0603_hand_solder, F.Cu at (151.4, 86.5)
- added D12: APA102-2020, tiny_pov_footprints:LED-APA102-2020, F.Cu at (228.7, 96.7)
- added D13: APA102-2020, tiny_pov_footprints:LED-APA102-2020, F.Cu at (224.9, 96.7)
- added D14: APA102-2020, tiny_pov_footprints:LED-APA102-2020, F.Cu at (221.1, 96.7)
- added D15: APA102-2020, tiny_pov_footprints:LED-APA102-2020, F.Cu at (217.3, 96.7)
- added D16: APA102-2020, tiny_pov_footprints:LED-APA102-2020, F.Cu at (213.5, 96.7)
- added D17: APA102-2020, tiny_pov_footprints:LED-APA102-2020, F.Cu at (209.7, 96.7)
- added D18: APA102-2020, tiny_pov_footprints:LED-APA102-2020, F.Cu at (205.9, 96.7)
- added D19: APA102-2020, tiny_pov_footprints:LED-APA102-2020, F.Cu at (202.1, 96.7)
- added D20: APA102-2020, tiny_pov_footprints:LED-APA102-2020, F.Cu at (198.3, 96.7)
- added D21: APA102-2020, tiny_pov_footprints:LED-APA102-2020, F.Cu at (194.5, 96.7)
- added D22: APA102-2020, tiny_pov_footprints:LED-APA102-2020, F.Cu at (190.7, 96.7)
- added D23: APA102-2020, tiny_pov_footprints:LED-APA102-2020, F.Cu at (186.9, 96.7)
- added D24: APA102-2020, tiny_pov_footprints:LED-APA102-2020, F.Cu at (183.1, 96.7)
- added D25: APA102-2020, tiny_pov_footprints:LED-APA102-2020, F.Cu at (179.3, 96.7)
- added D26: APA102-2020, tiny_pov_footprints:LED-APA102-2020, F.Cu at (175.5, 96.7)
- added D27: APA102-2020, tiny_pov_footprints:LED-APA102-2020, F.Cu at (171.7, 96.7)
- added D28: APA102-2020, tiny_pov_footprints:LED-APA102-2020, F.Cu at (167.9, 96.7)
- added D29: APA102-2020, tiny_pov_footprints:LED-APA102-2020, F.Cu at (164.1, 96.7)
- added D30: APA102-2020, tiny_pov_footprints:LED-APA102-2020, F.Cu at (160.3, 96.7)
- added D31: APA102-2020, tiny_pov_footprints:LED-APA102-2020, F.Cu at (156.5, 96.7)
- added D32: APA102-2020, tiny_pov_footprints:LED-APA102-2020, F.Cu at (152.7, 96.7)
- added D33: APA102-2020, tiny_pov_footprints:LED-APA102-2020, F.Cu at (148.9, 96.7)
- added D34: APA102-2020, tiny_pov_footprints:LED-APA102-2020, F.Cu at (145.1, 96.7)
- added D35: APA102-2020, tiny_pov_footprints:LED-APA102-2020, F.Cu at (141.3, 96.7)
- added D36: APA102-2020, tiny_pov_footprints:LED-APA102-2020, F.Cu at (137.5, 96.7)
- added D37: APA102-2020, tiny_pov_footprints:LED-APA102-2020, F.Cu at (133.7, 96.7)
- added D38: APA102-2020, tiny_pov_footprints:LED-APA102-2020, F.Cu at (129.9, 96.7)
- added D39: APA102-2020, tiny_pov_footprints:LED-APA102-2020, F.Cu at (126.1, 96.7)
- added D40: APA102-2020, tiny_pov_footprints:LED-APA102-2020, F.Cu at (122.3, 96.7)
- added D41: APA102-2020, tiny_pov_footprints:LED-APA102-2020, F.Cu at (118.5, 96.7)
- added D42: APA102-2020, tiny_pov_footprints:LED-APA102-2020, F.Cu at (114.7, 96.7)
- added D43: APA102-2020, tiny_pov_footprints:LED-APA102-2020, F.Cu at (110.9, 96.7)
- added D44: APA102-2020, tiny_pov_footprints:LED-APA102-2020, F.Cu at (107.1, 96.7)
- added D45: APA102-2020, tiny_pov_footprints:LED-APA102-2020, F.Cu at (103.3, 96.7)
- added D46: APA102-2020, tiny_pov_footprints:LED-APA102-2020, F.Cu at (99.5, 96.7)
- added D47: APA102-2020, tiny_pov_footprints:LED-APA102-2020, F.Cu at (95.7, 96.7)
- added D48: APA102-2020, tiny_pov_footprints:LED-APA102-2020, F.Cu at (91.9, 96.7)
- added D49: APA102-2020, tiny_pov_footprints:LED-APA102-2020, F.Cu at (88.1, 96.7)
- added D50: APA102-2020, tiny_pov_footprints:LED-APA102-2020, F.Cu at (84.3, 96.7)
- added D51: APA102-2020, tiny_pov_footprints:LED-APA102-2020, F.Cu at (80.5, 96.7)
- added D52: APA102-2020, tiny_pov_footprints:LED-APA102-2020, F.Cu at (76.7, 96.7)
- added D53: APA102-2020, tiny_pov_footprints:LED-APA102-2020, F.Cu at (72.9, 96.7)
- added D54: APA102-2020, tiny_pov_footprints:LED-APA102-2020, F.Cu at (69.1, 96.7)
- added D55: APA102-2020, tiny_pov_footprints:LED-APA102-2020, F.Cu at (65.3, 96.7)
- added D56: APA102-2020, tiny_pov_footprints:LED-APA102-2020, F.Cu at (61.5, 96.7)
- added D57: APA102-2020, tiny_pov_footprints:LED-APA102-2020, F.Cu at (57.7, 96.7)
- added D58: APA102-2020, tiny_pov_footprints:LED-APA102-2020, F.Cu at (53.9, 96.7)
- added D59: APA102-2020, tiny_pov_footprints:LED-APA102-2020, F.Cu at (50.1, 96.7)
- added D60: APA102-2020, tiny_pov_footprints:LED-APA102-2020, F.Cu at (46.3, 96.7)
- added D61: APA102-2020, tiny_pov_footprints:LED-APA102-2020, F.Cu at (42.5, 96.7)
- added D62: APA102-2020, tiny_pov_footprints:LED-APA102-2020, F.Cu at (38.7, 96.7)
- added D63: APA102-2020, tiny_pov_footprints:LED-APA102-2020, F.Cu at (34.9, 96.7)
- added D64: APA102-2020, tiny_pov_footprints:LED-APA102-2020, F.Cu at (31.1, 96.7)
- added J2: SdHolder, tiny_pov_footprints:microSD, B.Cu at (151.8, 91.7)
- added L1: 6.8uH, tiny_pov_footprints:L_0603_hand_solder, F.Cu at (153.7, 103.5)
- added R1: 10k, tiny_pov_footprints:R_0603_hand_solder, B.Cu at (142.6, 94.2)
- added R2: 47k, tiny_pov_footprints:R_0603_hand_solder, B.Cu at (142.6, 90.7)
- added R3: 47k, tiny_pov_footprints:R_0603_hand_solder, B.Cu at (142.6, 92.4)
- added R4: 47k, tiny_pov_footprints:R_0603_hand_solder, B.Cu at (142.6, 89.0)
- added TP1: TestPoint, tiny_pov_footprints:TestPoint_Pad, B.Cu at (136.9, 92.8)
- added TP2: TestPoint, tiny_pov_footprints:TestPoint_Pad, B.Cu at (133.9, 92.8)
- added TP3: TestPoint, tiny_pov_footprints:TestPoint_Pad, B.Cu at (163.3, 93.3)
- added TP4: TestPoint, tiny_pov_footprints:TestPoint_Pad, B.Cu at (160.3, 90.3)
- added TP5: TestPoint, tiny_pov_footprints:TestPoint_Pad, B.Cu at (163.3, 90.3)
- added U3: STM32G030J6Mx, tiny_pov_footprints:STM32_SO_8N, F.Cu at (146.9, 87.7)
- C1: value 100 uF -> ? uF; footprint tiny_pov_footprints:C_0402_hand_solder -> tiny_pov_footprints:C_polarized_TH; moved to B.Cu
- C2: footprint tiny_pov_footprints:C_0402_hand_solder -> tiny_pov_footprints:C_0603_hand_solder
- U1: value AH1806W -> AP63203WU; footprint tiny_pov_footprints:SC-59_Handsoldering -> tiny_pov_footprints:TSOT-23-6_HandSoldering
- U2: value STM32G030J6Mx -> AH1806W; footprint tiny_pov_footprints:STM32_SO_8N -> tiny_pov_footprints:SC-59_Handsoldering; moved to B.Cu
- moved D11 149.4 mm to (232.5, 96.7)
- moved D10 149.2 mm to (236.3, 96.7)
- moved D9 147.9 mm to (240.1, 96.7)
- moved D2 147.1 mm to (266.7, 96.7)
- moved D3 146.9 mm to (262.9, 96.7)
- moved D8 146.6 mm to (243.9, 96.7)
- moved D4 146.5 mm to (259.1, 96.7)
- moved D5 146.1 mm to (255.3, 96.7)
- moved D6 145.8 mm to (251.5, 96.7)
- moved D7 145.4 mm to (247.7, 96.7)
- moved D1 137.0 mm to (270.5, 96.7)
- moved JP1 22.4 mm to (153.7, 86.5), turned to -90 degrees
- moved J1 18.0 mm to (137.7, 101.1)
- moved U1 17.4 mm to (158.5, 102.5), turned to 180 degrees
- moved C1 13.6 mm to (165.4, 102.0), turned to -90 degrees
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Connections:
- C1 pad 1: Vdd -> N$29
- C2 pad 1: STM_RESET -> N$33
- C2 pad 2: GND -> N$34
- D11 pad 2: (no net) -> N$57
- D11 pad 3: (no net) -> N$58
- J1 pad 1: Vdd -> Vac_a
- J1 pad 2: GND -> Vac_b
- JP1 pad 1: STM_RESET -> HALL_DATA
- U1 pad 2: STM_RESET -> N$29
- U1 pad 3: GND -> N$29
- U2 pad 1: SD_SCK -> Vdd
- U2 pad 2: Vdd -> HALL_DATA
Routing:
- net Vdd: track 0.00 -> 496.4 mm, vias 0 -> 4
- net LED_CLK: track 0.00 -> 147.5 mm, vias 0 -> 3
- net LED_DATA: track 0.00 -> 146.7 mm, vias 0 -> 3
- net N$163: track 0.00 -> 38.8 mm
- net HALL_DATA: track 0.00 -> 29.7 mm, vias 0 -> 1
- net N$29: track 0.00 -> 28.5 mm, vias 0 -> 1
- net N$165: track 0.00 -> 24.7 mm
- net N$164: track 0.00 -> 23.1 mm
- net N$13: track 0.00 -> 13.9 mm
- net SD_SCK: track 0.00 -> 12.4 mm, vias 0 -> 1
- net SD_MOSI: track 0.00 -> 10.0 mm, vias 0 -> 1
- net Vac_a: track 0.00 -> 6.28 mm
- net Vac_b: track 0.00 -> 5.89 mm
- net GND: track 0.00 -> 4.60 mm, vias 0 -> 1
- net N$34: track 0.00 -> 4.47 mm
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- added copper zone on B.Cu, net GND
- added copper zone on F.Cu, net GND
Other:
- board outline added: 250 x 30.9 mm
- board text added: ":)"
- board text added: "TinyPOV v1.0"
- board text added: "www.michael-crum.com/tiny-pov"

Commit message: Iterated board layout
Parts:
- BR1, U1: moved to B.Cu
- R1, R2, R3, R4: moved to F.Cu
- moved TP2 52.0 mm to (183.5, 108.2)
- moved TP1 51.9 mm to (186.5, 108.2)
- moved TP4 24.9 mm to (177.5, 108.2)
- moved TP3 22.7 mm to (180.5, 108.2)
- moved TP5 21.1 mm to (174.5, 108.2)
- moved C4 18.7 mm to (143.8, 113.8), turned to 180 degrees
- moved C3 17.0 mm to (147.8, 111.5), turned to 0 degrees
- moved C6 16.1 mm to (143.1, 100.2), turned to 180 degrees
- moved C1 16.0 mm to (151.3, 109.5), turned to 0 degrees
- moved JP1 15.1 mm to (161.8, 99.2)
- moved U1 14.9 mm to (149.0, 114.0), turned to 0 degrees
- moved L1 14.5 mm to (147.8, 116.8)
- moved U2 12.3 mm to (162.0, 99.2), turned to 0 degrees
- moved U3 11.5 mm to (150.5, 98.6), turned to 0 degrees
- moved C2 10.2 mm to (153.2, 115.0), turned to 90 degrees
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Connections:
- net N$100 renamed apa_led_31_32_SD
- net N$101 renamed apa_led_32_33_CK
- net N$102 renamed apa_led_32_33_SD
- net N$103 renamed apa_led_33_34_CK
- net N$104 renamed apa_led_33_34_SD
- net N$105 renamed apa_led_34_35_CK
- net N$106 renamed apa_led_34_35_SD
- net N$107 renamed apa_led_35_36_CK
- net N$108 renamed apa_led_35_36_SD
- net N$109 renamed apa_led_36_37_CK
- net N$110 renamed apa_led_36_37_SD
- net N$111 renamed apa_led_37_38_CK
- net N$112 renamed apa_led_37_38_SD
- net N$113 renamed apa_led_38_39_CK
- net N$114 renamed apa_led_38_39_SD
- net N$115 renamed apa_led_39_40_CK
- net N$116 renamed apa_led_39_40_SD
- net N$117 renamed apa_led_40_41_CK
- net N$118 renamed apa_led_40_41_SD
- net N$119 renamed apa_led_41_42_CK
- net N$120 renamed apa_led_41_42_SD
- net N$121 renamed apa_led_42_43_CK
- net N$122 renamed apa_led_42_43_SD
- net N$123 renamed apa_led_43_44_CK
- net N$124 renamed apa_led_43_44_SD
- net N$125 renamed apa_led_44_45_CK
- net N$126 renamed apa_led_44_45_SD
- net N$127 renamed apa_led_45_46_CK
- net N$128 renamed apa_led_45_46_SD
- net N$129 renamed apa_led_46_47_CK
- net N$13 renamed SD_CS
- net N$130 renamed apa_led_46_47_SD
- net N$131 renamed apa_led_47_48_CK
- net N$132 renamed apa_led_47_48_SD
- net N$133 renamed apa_led_48_49_CK
- net N$134 renamed apa_led_48_49_SD
- net N$135 renamed apa_led_49_50_CK
- net N$136 renamed apa_led_49_50_SD
- net N$137 renamed apa_led_50_51_CK
- net N$138 renamed apa_led_50_51_SD
- net N$139 renamed apa_led_51_52_CK
- net N$140 renamed apa_led_51_52_SD
- net N$141 renamed apa_led_52_53_CK
- net N$142 renamed apa_led_52_53_SD
- net N$143 renamed apa_led_53_54_CK
- net N$144 renamed apa_led_53_54_SD
- net N$145 renamed apa_led_54_55_CK
- net N$146 renamed apa_led_54_55_SD
- net N$147 renamed apa_led_55_56_CK
- net N$148 renamed apa_led_55_56_SD
- net N$149 renamed apa_led_56_57_CK
- net N$150 renamed apa_led_56_57_SD
- net N$151 renamed apa_led_57_58_CK
- net N$152 renamed apa_led_57_58_SD
- net N$153 renamed apa_led_58_59_CK
- net N$154 renamed apa_led_58_59_SD
- net N$155 renamed apa_led_59_60_CK
- net N$156 renamed apa_led_59_60_SD
- net N$157 renamed apa_led_60_61_CK
- net N$158 renamed apa_led_60_61_SD
- net N$159 renamed apa_led_61_62_CK
- net N$160 renamed apa_led_61_62_SD
- net N$161 renamed apa_led_62_63_CK
- net N$162 renamed apa_led_62_63_SD
- net N$29 renamed V_rect_plus
- net N$33 renamed BST
- net N$34 renamed SW
- net N$37 renamed apa_led_0_1_CK
- net N$38 renamed apa_led_0_1_SD
- net N$39 renamed apa_led_1_2_CK
- net N$40 renamed apa_led_1_2_SD
- net N$41 renamed apa_led_2_3_CK
- net N$42 renamed apa_led_2_3_SD
- net N$43 renamed apa_led_3_4_CK
- net N$44 renamed apa_led_3_4_SD
- net N$45 renamed apa_led_4_5_CK
- net N$46 renamed apa_led_4_5_SD
- net N$47 renamed apa_led_5_6_CK
- net N$48 renamed apa_led_5_6_SD
- net N$49 renamed apa_led_6_7_CK
- net N$50 renamed apa_led_6_7_SD
- net N$51 renamed apa_led_7_8_CK
- net N$52 renamed apa_led_7_8_SD
- net N$53 renamed apa_led_8_9_CK
- net N$54 renamed apa_led_8_9_SD
- net N$55 renamed apa_led_9_10_CK
- net N$56 renamed apa_led_9_10_SD
- net N$57 renamed apa_led_10_11_CK
- net N$58 renamed apa_led_10_11_SD
- net N$59 renamed apa_led_11_12_CK
- net N$60 renamed apa_led_11_12_SD
- net N$61 renamed apa_led_12_13_CK
- net N$62 renamed apa_led_12_13_SD
- net N$63 renamed apa_led_13_14_CK
- net N$64 renamed apa_led_13_14_SD
- net N$65 renamed apa_led_14_15_CK
- net N$66 renamed apa_led_14_15_SD
- net N$67 renamed apa_led_15_16_CK
- net N$68 renamed apa_led_15_16_SD
- net N$69 renamed apa_led_16_17_CK
- net N$70 renamed apa_led_16_17_SD
- net N$71 renamed apa_led_17_18_CK
- net N$72 renamed apa_led_17_18_SD
- net N$73 renamed apa_led_18_19_CK
- net N$74 renamed apa_led_18_19_SD
- net N$75 renamed apa_led_19_20_CK
- net N$76 renamed apa_led_19_20_SD
- net N$77 renamed apa_led_20_21_CK
- net N$78 renamed apa_led_20_21_SD
- net N$79 renamed apa_led_21_22_CK
- net N$80 renamed apa_led_21_22_SD
- net N$81 renamed apa_led_22_23_CK
- net N$82 renamed apa_led_22_23_SD
- net N$83 renamed apa_led_23_24_CK
- net N$84 renamed apa_led_23_24_SD
- net N$85 renamed apa_led_24_25_CK
- net N$86 renamed apa_led_24_25_SD
- net N$87 renamed apa_led_25_26_CK
- net N$88 renamed apa_led_25_26_SD
- net N$89 renamed apa_led_26_27_CK
- net N$90 renamed apa_led_26_27_SD
- net N$91 renamed apa_led_27_28_CK
- net N$92 renamed apa_led_27_28_SD
- net N$93 renamed apa_led_28_29_CK
- net N$94 renamed apa_led_28_29_SD
- net N$95 renamed apa_led_29_30_CK
- net N$96 renamed apa_led_29_30_SD
- net N$97 renamed apa_led_30_31_CK
- net N$98 renamed apa_led_30_31_SD
- net N$99 renamed apa_led_31_32_CK
- J2 pad 3: N$164 -> SD_MOSI
- J2 pad 5: N$163 -> SD_SCK
- J2 pad 7: N$165 -> SD_MISO
- R2 pad 1: N$163 -> SD_SCK
- R2 pad 2: SD_SCK -> Vdd
- R3 pad 1: N$164 -> SD_MOSI
- R3 pad 2: SD_MOSI -> Vdd
- R4 pad 1: N$165 -> SD_MISO
- R4 pad 2: SD_MISO -> Vdd
- TP3 pad 1: N$163 -> SD_SCK
- TP4 pad 1: N$164 -> SD_MOSI
- TP5 pad 1: N$165 -> SD_MISO
Routing:
- net GND: track 4.60 -> 199.5 mm, vias 1 -> 131
- net SD_MOSI: track 10.0 -> 52.0 mm, vias 1 -> 2
- net SD_MISO: track 3.13 -> 44.4 mm, vias 1 -> 3
- net SD_SCK: track 12.4 -> 52.1 mm
- net N$163: track 38.8 -> 0.00 mm
- net Vdd: track 496.4 -> 463.9 mm, vias 4 -> 5
- net N$165: track 24.7 -> 0.00 mm
- net N$164: track 23.1 -> 0.00 mm
- net LED_CLK: track 147.5 -> 126.3 mm, vias 3 -> 2
- net LED_DATA: track 146.7 -> 125.8 mm, vias 3 -> 2
- net V_rect_plus: track 28.5 -> 15.5 mm, vias 1 -> 0
- net HALL_DATA: track 29.7 -> 19.5 mm, vias 1 -> 2
- net SW: track 4.47 -> 10.4 mm, vias 0 -> 1
- net SD_CS: track 13.9 -> 8.71 mm, vias 0 -> 1
- net Vac_a: track 6.28 -> 3.53 mm
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Other:
- board size 250 x 30.9 mm -> 250 x 30.5 mm
- board text added: "michael-crum.com/tiny-pov"
- board text removed: ":)"
- board text removed: "www.michael-crum.com/tiny-pov"

Commit message: v1 board ordered
Other:
- board text added: ":)"
Changed lines of the file:
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@@
   (gr_line (start 127.687659 100) (end 30 100)
     (stroke (width 0.2) (type solid)) (layer "Edge.Cuts"))
+  (gr_text ":)" (at 271 105.75) (layer "B.SilkS")
+    (effects (font (size 1.5 1.5) (thickness 0.3) bold) (justify left bottom))
+  )
   (gr_text "michael-crum.com/tiny-pov" (at 63.78 105.94) (layer "B.SilkS")
     (effects (font (size 1.5 1.5) (thickness 0.3) bold) (justify left bottom mirror))
