File: HARDWARE/tiny_pov_arm/tiny_pov_arm.kicad_pcb (KiCad board)
At the start: 2 copper layers, 250 x 30.5 mm, 87 parts, among them J1 Conn_01x02_Socket, J2 SdHolder, U1 AP63203WU, U2 AH1806W, U3 STM32G030J6Mx

Commit message: Changed apa102 to correct footprint, changed STM32 pinout to allow for SPI
Parts:
- removed C6: 100 nF, tiny_pov_footprints:C_0603_hand_solder
- D1, D10, D11, D12, D13, D14, D15, D16, D17, D18, D19, D2, D20, D21, D22, D23, D24, D25, D26, D27, D28, D29, D3, D30, D31, D32, D33, D34, D35, D36, D37, D38, D39, D4, D40, D41, D42, D43, D44, D45, D46, D47, D48, D49, D5, D50, D51, D52, D53, D54, D55, D56, D57, D58, D59, D6, D60, D61, D62, D63, D64, D7, D8, D9: footprint tiny_pov_footprints:LED-APA102-2020 -> tiny_pov_footprints:LED_APA-102-2020-256-8
Connections:
- JP1 pad 1: HALL_DATA -> LED_CLK
- U3 pad 4: HALL_DATA -> LED_CLK
- U3 pad 7: LED_CLK -> HALL_DATA
Routing:
- net HALL_DATA: track 19.5 -> 8.95 mm, vias 2 -> 1
- net LED_CLK: track 126.3 -> 134.0 mm, vias 2 -> 4

Commit message: Arm board v1.1
Parts:
- removed JP1: SolderJumper_2_Open, tiny_pov_footprints:SolderJumper
- removed TP1, TP2, TP3, TP4, TP5: TestPoint, tiny_pov_footprints:TestPoint_Pad
- added C10: 22 uF, tiny_pov_footprints:C_0603_hand_solder, B.Cu at (160.4, 108.2)
- added C11: 22 uF, tiny_pov_footprints:C_0603_hand_solder, B.Cu at (163.8, 106.8)
- added C12: 22 uF, tiny_pov_footprints:C_0603_hand_solder, B.Cu at (163.8, 105.2)
- added C13: 22 uF, tiny_pov_footprints:C_0603_hand_solder, B.Cu at (163.8, 103.8)
- added C6: 100 nF, tiny_pov_footprints:C_0603_hand_solder, F.Cu at (158.5, 104.5)
- added C7: 22 uF, tiny_pov_footprints:C_0603_hand_solder, B.Cu at (160.4, 103.8)
- added C8: 22 uF, tiny_pov_footprints:C_0603_hand_solder, B.Cu at (160.4, 105.2)
- added C9: 22 uF, tiny_pov_footprints:C_0603_hand_solder, B.Cu at (160.4, 106.8)
- C1: value ? uF -> 22 uF; footprint tiny_pov_footprints:C_polarized_TH -> tiny_pov_footprints:C_0603_hand_solder
- C2: value 100 nF -> 22 uF; moved to B.Cu
- C3, C4: moved to B.Cu
- C5: value 100 uF -> 22 uF; footprint tiny_pov_footprints:C_polarized_TH -> tiny_pov_footprints:C_0603_hand_solder
- U1: moved to F.Cu
- moved U2 37.3 mm to (124.8, 96.8)
- moved L1 16.2 mm to (160.4, 106.8), turned to 0 degrees
- moved R3 11.4 mm to (150.9, 89.0), turned to -90 degrees
- moved R1 10.7 mm to (152.4, 89.0), turned to 90 degrees
- moved R4 10.4 mm to (146.5, 88.9), turned to -90 degrees
- moved C4 9.92 mm to (152.9, 110.0)
- moved U1 9.69 mm to (155.7, 107.0)
- moved R2 8.80 mm to (148.7, 89.0), turned to -90 degrees
- moved C3 8.67 mm to (156.3, 110.0)
- moved J1 7.33 mm to (137.6, 106.4), turned to 180 degrees
- moved BR1 7.30 mm to (145.3, 106.9), turned to 180 degrees
- moved C2 7.15 mm to (156.3, 108.5), turned to 0 degrees
- moved J2 5.35 mm to (150.0, 93.5)
- moved U3 5.22 mm to (150.0, 93.4)
- moved D1 5.00 mm to (269.0, 100.0)
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Connections:
- C2 pad 1: BST -> V_rect_plus
- C2 pad 2: SW -> GND
- C3 pad 1: Vdd -> V_rect_plus
- C4 pad 1: Vdd -> V_rect_plus
- C5 pad 1: Vdd -> V_rect_plus
- U3 pad 5: SD_MOSI -> SD_MISO
- U3 pad 6: LED_DATA -> SD_MOSI
- U3 pad 8: SD_MISO -> LED_DATA
Routing:
- net GND: track 199.5 -> 3.26 mm, vias 131 -> 77
- net SD_SCK: track 52.1 -> 3.98 mm, vias 1 -> 2
- net SD_MOSI: track 52.0 -> 6.68 mm
- net Vdd: track 464.3 -> 423.5 mm, vias 5 -> 8
- net SD_MISO: track 44.4 -> 11.2 mm, vias 3 -> 2
- net HALL_DATA: track 8.95 -> 31.2 mm
- net SD_CS: track 8.71 -> 0.00 mm
- net LED_CLK: track 134.0 -> 126.7 mm, vias 4 -> 0
- net V_rect_plus: track 15.5 -> 22.0 mm, vias 0 -> 2
- net SW: track 10.4 -> 4.56 mm, vias 1 -> 0
- net Vac_a: track 3.53 -> 5.08 mm
- net BST: track 3.03 -> 1.59 mm, vias 1 -> 0
- net LED_DATA: track 125.8 -> 124.7 mm, vias 2 -> 0
- net Vac_b: track 4.78 -> 4.06 mm
Other:
- board text added: "Tiny POV v1.1"
- board text added: "michael-crum.com/tiny-pov/"
- board text removed: "TinyPOV v1.0"
- board text removed: "michael-crum.com/tiny-pov"
